File: fpga_board.kicad_sch (KiCad schematic)
At the start: 206 parts, among them Q1 2N7002PW, Q2 2N7002PW, Q3 2N7002PW, Q4 2N7002PW, Q5 2N7002PW, Q6 2N7002PW, SW1 1TS028A-1300-0600-CT, U1 LFE5U-45F-6BG256C, U10 TLV62569DRL, U2 CYUSB3014-BZXC, U3 TLV62569DRL, U5 MT41K256M16TW-093:P, U6 MT41K256M16TW-093:P, U7 TLV62569DRL, U8 TLV62569DRL, U9 TLV62569DRL, X1 XO32, Y1 Crystal_GND24

Commit message: Switched VREF testpoint to F.Cu and removed Testpoints from BOM
Parts:
- TP1, TP2, TP3, TP4, TP5, TP6, TP7: now left out of the parts list
Changed lines of the file:
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@@
 		(unit 1)
 		(exclude_from_sim no)
-		(in_bom yes)
+		(in_bom no)
 		(on_board yes)
 		(dnp no)
@@
 		(unit 1)
 		(exclude_from_sim no)
-		(in_bom yes)
+		(in_bom no)
 		(on_board yes)
 		(dnp no)
@@
 		(unit 1)
 		(exclude_from_sim no)
-		(in_bom yes)
+		(in_bom no)
 		(on_board yes)
 		(dnp no)
@@
 		(unit 1)
 		(exclude_from_sim no)
-		(in_bom yes)
+		(in_bom no)
 		(on_board yes)
 		(dnp no)
@@
 		(unit 1)
 		(exclude_from_sim no)
-		(in_bom yes)
+		(in_bom no)
 		(on_board yes)
 		(dnp no)
@@
 		(unit 1)
 		(exclude_from_sim no)
-		(in_bom yes)
+		(in_bom no)
 		(on_board yes)
 		(dnp no)
@@
 		(unit 1)
 		(exclude_from_sim no)
-		(in_bom yes)
+		(in_bom no)
 		(on_board yes)
 		(dnp no)
